File: Photon/V1/PCB/DisplayStick.brd (EAGLE design)
At the start: 50 x 130 mm, 71 parts

Commit message: Added links for touch and sd card chip selects. Removed upper J10 4 pin connector so it's more obvious which connector the display should go into.
Bumped to V1.1
Parts:
- removed JP10: (no value), SparkFun-Connectors:1X04
- added R5, R6: (no value), SparkFun-Resistors:1206
- R1, R3: value (none) -> 10k
- R2: value (none) -> 0R
- moved LOGO1 29.2 mm to (24.9, 5.71)
- moved R4 5.08 mm to (11.7, 127.0)
- moved R2 0.32 mm to (26.4, 53.0)
Connections:
- net A0: now also R6.2
- net A1: now also R5.2
- net DISPLAY_MISO: no longer JP10.3
- net DISPLAY_MOSI: no longer JP10.2
- net DISPLAY_SCK: no longer JP10.4
- net RX: now also R7.2
- net SD_CS: now also R6.1; no longer JP10.1
- net TOUCH_CS: now also R5.1
- net WKP: no longer R7.2
Routing:
- net A0: track 12.9 -> 120.0 mm
- net RX: track 12.9 -> 45.3 mm, vias 0 -> 1
- net WKP: track 42.8 -> 13.1 mm, vias 1 -> 0
- net SD_CS: track 5.36 -> 24.1 mm
- net DISPLAY_MISO: track 180.4 -> 172.5 mm, vias 2 -> 1
- net A1: track 12.9 -> 20.0 mm
- net DISPLAY_SCK: track 186.7 -> 180.5 mm, vias 1 -> 0
- net DISPLAY_MOSI: track 191.9 -> 186.3 mm
- net TOUCH_CS: track 10.5 -> 14.8 mm
- net 3.3V: track 187.4 -> 184.6 mm
Other:
- board text added: "-- Display"
- board text added: "10k"
- board text added: "21 Aug 2017"
- board text added: "CLK"
- board text added: "CS (A2)"
- board text added: "D/C (D2)"
- board text added: "D_CS"
- board text added: "IRQ->WKP"
- board text added: "LED"
- board text added: "MISO/DO"
- board text added: "MOSI/DIN"
- board text added: "RESET (D3)"
- board text added: "SD_CS"
- board text added: "SD_CS Pullup"
- board text added: "SD_CS->A0"
- board text added: "T_CLK"
- board text added: "T_CS"
- board text added: "T_CS->A1"
- board text added: "T_DIN"
- board text added: "T_DO"
- board text added: "T_IRQ"
- board text added: "T_IRQ (RX)"
- board text added: "ThingySticks.com/DisplayStick/V1"
- board text added: "V1.1"
- board text added: "VCC"
- board text added: "https://github.com/ThingySticks/DisplayStick"
- board text removed: "5 May 2017"
- board text removed: "V1.0"
