File: Photon/V1/PCB/DisplayStick.sch (EAGLE design)
At the start: 71 parts

Commit message: Added links for touch and sd card chip selects. Removed upper J10 4 pin connector so it's more obvious which connector the display should go into.
Bumped to V1.1
Parts:
- removed JP10: (no value), SparkFun-Connectors:M04PTH
- added R5, R6: (no value), SparkFun-Resistors:RESISTOR1206
- R1, R3: value (none) -> 10k
- R2: value (none) -> 0R
Connections:
- net A0: now also R6.2
- net A1: now also R5.2
- net DISPLAY_MISO: no longer JP10.3
- net DISPLAY_MOSI: no longer JP10.2
- net DISPLAY_SCK: no longer JP10.4
- net RX: now also R7.2
- net SD_CS: now also R6.1; no longer JP10.1
- net TOUCH_CS: now also R5.1
- net WKP: no longer R7.2
Other:
- note added: "1.1"
- note added: "Stephen Harrison"
- moved on the sheet: R1, R2, R3
